Commit message: [thormang3_description] Update for Melodic

File: thormang3_description/urdf/thormang3.structure.arm.xacro (robot description, xacro)
@@ -1,5 +1,4 @@
 <?xml version="1.0"?>
 <robot xmlns:xacro="http://ros.org/wiki/xacro">
-    <xacro:property name="pi" value="3.141592654" />
     <xacro:property name="offset" value="0.0" />
     <xacro:macro name="thormang3_l_arm" params="parent">

File: thormang3_description/urdf/thormang3.structure.head.xacro (robot description, xacro)
@@ -1,5 +1,4 @@
 <?xml version="1.0"?>
 <robot xmlns:xacro="http://ros.org/wiki/xacro">
-    <xacro:property name="pi" value="3.141592654" />
     <xacro:macro name="thormang3_head" params="parent">
 	<!-- head yaw joint -->

File: thormang3_description/urdf/thormang3.structure.leg.xacro (robot description, xacro)
@@ -1,5 +1,4 @@
 <?xml version="1.0"?>
 <robot xmlns:xacro="http://ros.org/wiki/xacro">
-    <xacro:property name="pi" value="3.141592654" />
     <xacro:macro name="thormang3_l_leg" params="parent">
 	<!-- left hip yaw joint -->

File: thormang3_description/urdf/thormang3.xacro (robot description, xacro)
@@ -2,6 +2,4 @@
 <!-- Revolute-Revolute Manipulator -->
 <robot name="thormang3" xmlns:xacro="http://www.ros.org/wiki/xacro">
-  <!-- some parameters -->
-  <xacro:property name="pi" value="3.141592654" />
   <!-- Import all Gazebo-customization elements, including Gazebo colors -->
   <xacro:include filename="$(find thormang3_description)/urdf/thormang3.gazebo" />
