Commit message: [thormang3_description] Fix neck joints

File: thormang3_description/urdf/thormang3.structure.head.xacro (robot description, xacro)
@@ -3,5 +3,5 @@
     <xacro:macro name="thormang3_head" params="parent">
 	<!-- head yaw joint -->
-        <joint name="head_y" type="revolute">
+        <joint name="head_y" type="fixed">
           <axis xyz="0 0 1" />
           <origin xyz="0.0 0.0 0.229" rpy="0 0 0"/>
@@ -34,5 +34,5 @@
         </link>
 	<!-- head pitch joint -->
-        <joint name="head_p" type="revolute">
+        <joint name="head_p" type="fixed">
           <axis xyz="0 1 0" />
           <origin xyz="0.0 -0.045 0.039" rpy="0 0 0"/>
